File: PCB/BoomBox.kicad_pcb (KiCad board)
At the start: 2 copper layers, 28.6 x 77.4 mm, 4 parts, among them SW1 SW_Push, SW2 SW_Push, SW3 SW_Push, U1 XIAO-RP2040-DIP

Commit message: Add files via upload
Parts:
- moved SW3 5.05 mm to (107.3, 90.5)
- moved SW2 2.68 mm to (107.3, 71.4)
- moved SW1 0.35 mm to (107.3, 52.4)
Routing:
- net Net-(U1-GPIO4/MISO): track 61.2 -> 66.7 mm
- net GND: track 58.6 -> 62.6 mm
- net Net-(U1-GPIO2/SCK): track 63.7 -> 66.7 mm
Other:
- board size 28.6 x 77.4 mm -> 28.6 x 83.4 mm
Changed lines of the file:
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@@
 			(sketchdnponfab yes)
 			(crossoutdnponfab yes)
-			(subtractmaskfromsilk no)
+			(subtractmaskfromsilk yes)
 			(outputformat 1)
 			(mirror no)
 			(drillshape 0)
 			(scaleselection 1)
-			(outputdirectory "C:/Users/Rohan/Downloads/")
+			(outputdirectory "./")
 		)
 	)
@@
 	(footprint "Button_Switch_Keyboard:SW_Cherry_MX_1.00u_PCB"
 		(layer "F.Cu")
-		(at 107.315 52.07)
+		(at 107.315 52.42)
 		(descr "Cherry MX keyswitch, 1.00u, PCB mount, http://cherryamericas.com/wp-content/uploads/2014/12/mx_cat.pdf")
 		(tags "Cherry MX keyswitch 1.00u PCB")
@@
 	(footprint "Button_Switch_Keyboard:SW_Cherry_MX_1.00u_PCB"
 		(layer "F.Cu")
-		(at 107.315 85.4075)
+		(at 107.315 90.46)
 		(descr "Cherry MX keyswitch, 1.00u, PCB mount, http://cherryamericas.com/wp-content/uploads/2014/12/mx_cat.pdf")
 		(tags "Cherry MX keyswitch 1.00u PCB")
@@
 	(footprint "Button_Switch_Keyboard:SW_Cherry_MX_1.00u_PCB"
 		(layer "F.Cu")
-		(at 107.315 68.73875)
+		(at 107.315 71.42)
 		(descr "Cherry MX keyswitch, 1.00u, PCB mount, http://cherryamericas.com/wp-content/uploads/2014/12/mx_cat.pdf")
 		(tags "Cherry MX keyswitch 1.00u PCB")
@@
 	(gr_rect
 		(start 90.4875 23.8125)
-		(end 119.0625 101.203125)
+		(end 119.0625 107.203125)
 		(stroke
 			(width 0.05)
@@
 	)
 	(segment
-		(start 107.315 52.07)
-		(end 107.315 68.73875)
-		(width 0.2)
-		(layer "F.Cu")
-		(net 1)
-	)
-	(segment
-		(start 107.315 68.73875)
-		(end 107.315 85.4075)
+		(start 107.315 71.42)
+		(end 107.315 90.46)
 		(width 0.2)
 		(layer "F.Cu")
@@
 	)
 	(segment
+		(start 107.315 53.42)
+		(end 107.315 71.77)
+		(width 0.2)
+		(layer "F.Cu")
+		(net 1)
+	)
+	(segment
 		(start 100.965 54.61)
 		(end 100.965 37.61709)
@@
 	)
 	(segment
-		(start 100.965 71.27875)
-		(end 100.965 57.635184)
+		(start 113.39575 38.89375)
+		(end 111.91875 38.89375)
 		(width 0.2)
 		(layer "F.Cu")
@@
 	)
 	(segment
-		(start 105.914 52.686184)
+		(start 111.47844 27.67075)
+		(end 114.009376 27.67075)
+		(width 0.2)
+		(layer "F.Cu")
+		(net 3)
+	)
+	(segment
+		(start 105.914 53.036184)
 		(end 105.914 33.23519)
+		(width 0.2)
+		(layer "F.Cu")
+		(net 3)
+	)
+	(segment
+		(start 114.009376 27.67075)
+		(end 114.27075 27.932124)
 		(width 0.2)
 		(layer "F.Cu")
@@
 	)
 	(segment
+		(start 114.27075 27.932124)
+		(end 114.27075 38.01875)
+		(width 0.2)
+		(layer "F.Cu")
+		(net 3)
+	)
+	(segment
+		(start 100.965 57.985184)
+		(end 105.914 53.036184)
+		(width 0.2)
+		(layer "F.Cu")
+		(net 3)
+	)
+	(segment
 		(start 105.914 33.23519)
 		(end 111.47844 27.67075)
@@
 	)
 	(segment
-		(start 111.47844 27.67075)
-		(end 114.009376 27.67075)
+		(start 100.965 74.31)
+		(end 100.965 57.985184)
 		(width 0.2)
 		(layer "F.Cu")
@@
 	)
 	(segment
-		(start 113.39575 38.89375)
-		(end 111.91875 38.89375)
-		(width 0.2)
-		(layer "F.Cu")
-		(net 3)
-	)
-	(segment
-		(start 114.009376 27.67075)
-		(end 114.27075 27.932124)
-		(width 0.2)
-		(layer "F.Cu")
-		(net 3)
-	)
-	(segment
-		(start 100.965 57.635184)
-		(end 105.914 52.686184)
-		(width 0.2)
-		(layer "F.Cu")
-		(net 3)
-	)
-	(segment
-		(start 114.27075 27.932124)
-		(end 114.27075 38.01875)
-		(width 0.2)
-		(layer "F.Cu")
-		(net 3)
-	)
-	(segment
-		(start 106.756314 87.9475)
-		(end 108.716 85.987814)
+		(start 107.895314 89.059)
+		(end 108.716 89.879686)
 		(width 0.2)
 		(layer "F.Cu")
@@
 	)
 	(segment
-		(start 108.716 84.827186)
-		(end 107.895314 84.0065)
+		(start 108.716 70.839686)
+		(end 108.716 72.000314)
 		(width 0.2)
 		(layer "F.Cu")
@@
 	)
 	(segment
-		(start 107.895314 70.13975)
-		(end 108.716 69.319064)
+		(start 112.75375 36.35375)
+		(end 108.716 40.3915)
 		(width 0.2)
 		(layer "F.Cu")
@@
 	)
 	(segment
-		(start 108.716 68.158436)
-		(end 107.895314 67.33775)
+		(start 107.895314 72.821)
+		(end 107.895314 89)
 		(width 0.2)
 		(layer "F.Cu")
@@
 	)
 	(segment
-		(start 107.895314 67.33775)
-		(end 107.895314 53.471)
+		(start 106.756314 93)
+		(end 100.965 93)
 		(width 0.2)
 		(layer "F.Cu")
@@
 	)
 	(segment
-		(start 107.895314 53.471)
+		(start 108.716 91.040314)
+		(end 106.756314 93)
+		(width 0.2)
+		(layer "F.Cu")
+		(net 4)
+	)
+	(segment
+		(start 107.895314 70.019)
+		(end 108.716 70.839686)
+		(width 0.2)
+		(layer "F.Cu")
+		(net 4)
+	)
+	(segment
+		(start 108.716 52.5)
 		(end 108.716 52.650314)
 		(width 0.2)
@@
 	)
 	(segment
-		(start 108.716 69.319064)
-		(end 108.716 68.158436)
+		(start 108.716 53.679314)
+		(end 108.716 52.5)
 		(width 0.2)
 		(layer "F.Cu")
@@
 	)
 	(segment
-		(start 108.716 85.987814)
-		(end 108.716 84.827186)
+		(start 108.716 40.3915)
+		(end 108.716 52.5)
 		(width 0.2)
 		(layer "F.Cu")
@@
 	)
 	(segment
-		(start 100.965 87.9475)
-		(end 106.756314 87.9475)
+		(start 108.716 72.000314)
+		(end 107.895314 72.821)
 		(width 0.2)
 		(layer "F.Cu")
@@
 	)
 	(segment
-		(start 108.716 52.650314)
-		(end 108.716 40.3915)
+		(start 108.716 89.879686)
+		(end 108.716 91.040314)
 		(width 0.2)
 		(layer "F.Cu")
@@
 	)
 	(segment
-		(start 108.716 40.3915)
-		(end 112.75375 36.35375)
+		(start 107.895314 54.5)
+		(end 107.895314 70.369)
 		(width 0.2)
 		(layer "F.Cu")
@@
 	)
 	(segment
-		(start 107.895314 84.0065)
-		(end 107.895314 70.13975)
-		(width 0.2)
-		(layer "F.Cu")
+		(start 107.895314 54.5)
+		(end 108.716 53.679314)
+		(width 0.2)
+		(layer "F.Cu")
